Commit message: Integrated the Ultrasound Image generation function with the simulator

File: catkin_ws/src/BTP/Franka_Emika/franka_discription/robots/hand.xacro (robot description, xacro)
@@ -62,4 +62,23 @@
       </inertial>
     </link>
+    <!-- <link name="${ns}_probe">
+      <visual>
+        <origin xyz="0 0 0" rpy="0 0 ${pi}"/>
+        <geometry>
+          <mesh filename="package://franka_description/meshes/visual/Ultrasonic-Probe.stl" scale="0.0007 0.0007 0.0007"/>
+        </geometry>
+      </visual>
+      <collision>
+        <origin xyz="0 0 0" rpy="0 0 ${pi}"/>
+        <geometry>
+          <mesh filename="package://franka_description/meshes/collision/Ultrasonic-Probe.stl" scale="0.0007 0.0007 0.0007"/>
+        </geometry>
+      </collision>
+      <inertial>
+        <origin xyz="0 0 0" rpy="0 0 ${pi}"/>
+        <mass value="0.2"/>
+        <inertia ixx="0.1" ixy="0.0" ixz="0.0" iyy="0.1" iyz="0.0" izz="0.1"/>
+      </inertial>
+    </link> -->
     <joint name="${ns}_finger_joint1" type="prismatic">
       <parent link="${ns}_hand"/>
@@ -77,4 +96,9 @@
       <mimic joint="${ns}_finger_joint1" />
     </joint>
+    <!-- <joint name="${ns}_probe_joint" type="fixed">
+      <parent link="${ns}_hand"/>
+      <child link="${ns}_probe"/>
+      <origin xyz="-0.02 0.025 0.15" rpy="1.57089 -0.002766 1.53752"/>
+    </joint> -->
   </xacro:macro>
 </robot>

File: catkin_ws/src/BTP/Franka_Emika/franka_discription/robots/panda.gazebo.xacro (robot description, xacro)
@@ -74,4 +74,9 @@
             <mu2>0.2</mu2>
         </gazebo>
+        <gazebo reference="${robot_name}_probe">
+            <material>Gazebo/Red</material>
+            <mu1>0.2</mu1>
+            <mu2>0.2</mu2>
+        </gazebo>
     </xacro:macro>
 </robot>
