Commit message: Redefined the reward function and completed the training code

File: catkin_ws/src/BTP/Franka_Emika/franka_discription/robots/panda.gazebo.xacro (robot description, xacro)
@@ -7,4 +7,15 @@
             <mu1>0.2</mu1>
             <mu2>0.2</mu2>
+            <!-- <sensor name="contact_sensor" type="contact" always_on="true" update_rate="100.0">
+                <contact>
+                    <collision> __default__</collision>
+                </contact>
+                <plugin name="plugin_1" filename="libgazebo_ros_bumper.so">
+                    <alwaysOn>true</alwaysOn>
+                    <updateRate>100.0</updateRate>
+                    <frameName>world</frameName>
+                    <bumperTopicName>panda_contact/link0</bumperTopicName>
+                </plugin>
+            </sensor> -->
         </gazebo>
         <!-- Link1 -->
@@ -74,9 +85,4 @@
             <mu2>0.2</mu2>
         </gazebo>
-        <gazebo reference="${robot_name}_probe">
-            <material>Gazebo/Red</material>
-            <mu1>0.2</mu1>
-            <mu2>0.2</mu2>
-        </gazebo>
     </xacro:macro>
 </robot>
